File: untitled.sch (EAGLE design)
At the start: 13 parts, among them IC1 NE555D

Commit message: Prepared for prodution
Parts:
- PR1: value (none) -> 10K
- Q1: value (none) -> MOSFET-N; device IGBT:IGBTTO252_STM -> mosfet_to252:MOSFET-N
- renumbered R3 to PR1
Connections:
- net GND: now also Q1.S; no longer Q1.E
- net N$11: now also Q1.D; no longer Q1.C
Changed lines of the file:
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@@
 <part name="C2" library="rcl" deviceset="C-EU" device="C1206" value="100n"/>
 <part name="C3" library="rcl" deviceset="C-EU" device="C0603" value="10n"/>
-<part name="Q1" library="IGBT" deviceset="IGBT" device="TO252_STM"/>
-<part name="R3" library="pot" deviceset="3RP/1610N" device=""/>
+<part name="Q1" library="mosfet_to252" deviceset="MOSFET-N" device=""/>
+<part name="PR1" library="pot" deviceset="3RP/1610N" device="" value="10K"/>
 <part name="JP1" library="pinhead" deviceset="PINHD-1X2" device="" value="ZAS"/>
 <part name="JP2" library="pinhead" deviceset="PINHD-1X2" device="" value="OUT"/>
@@
 </plain>
 <instances>
-<instance part="IC1" gate="A" x="43.18" y="50.8"/>
-<instance part="D1" gate="G$1" x="17.78" y="55.88"/>
+<instance part="IC1" gate="A" x="43.18" y="50.8" smashed="yes">
+<attribute name="NAME" x="36.322" y="61.468" size="1.778" layer="95"/>
+<attribute name="VALUE" x="41.402" y="61.341" size="1.778" layer="96"/>
+</instance>
+<instance part="D1" gate="G$1" x="17.78" y="55.88" smashed="yes">
+<attribute name="NAME" x="11.684" y="54.8386" size="1.778" layer="95"/>
+<attribute name="VALUE" x="20.32" y="53.5686" size="1.778" layer="96"/>
+</instance>
 <instance part="D2" gate="G$1" x="17.78" y="66.04" rot="R180"/>
-<instance part="R1" gate="G$1" x="63.5" y="48.26" rot="R90"/>
+<instance part="R1" gate="G$1" x="63.5" y="48.26" smashed="yes" rot="R90">
+<attribute name="NAME" x="65.024" y="49.2506" size="1.778" layer="95"/>
+<attribute name="VALUE" x="65.024" y="46.99" size="1.778" layer="96"/>
+</instance>
 <instance part="R2" gate="G$1" x="68.58" y="58.42"/>
-<instance part="C1" gate="G$1" x="20.32" y="48.26"/>
+<instance part="C1" gate="G$1" x="20.32" y="48.26" smashed="yes">
+<attribute name="NAME" x="14.224" y="48.387" size="1.778" layer="95"/>
+<attribute name="VALUE" x="13.462" y="43.561" size="1.778" layer="96"/>
+</instance>
 <instance part="C2" gate="G$1" x="0" y="76.2"/>
-<instance part="C3" gate="G$1" x="25.4" y="45.72"/>
-<instance part="Q1" gate="G$1" x="76.2" y="60.96"/>
-<instance part="R3" gate="G$1" x="25.4" y="60.96"/>
+<instance part="C3" gate="G$1" x="25.4" y="45.72" smashed="yes">
+<attribute name="NAME" x="26.924" y="46.101" size="1.778" layer="95"/>
+<attribute name="VALUE" x="25.654" y="41.529" size="1.778" layer="96"/>
+</instance>
+<instance part="Q1" gate="G$1" x="76.2" y="60.96" smashed="yes">
+<attribute name="VALUE" x="82.55" y="57.658" size="1.778" layer="96"/>
+<attribute name="NAME" x="82.55" y="59.944" size="1.778" layer="95"/>
+</instance>
+<instance part="PR1" gate="G$1" x="25.4" y="60.96" smashed="yes">
+<attribute name="NAME" x="22.352" y="63.119" size="1.778" layer="95" rot="R180"/>
+<attribute name="VALUE" x="22.098" y="60.706" size="1.778" layer="96" rot="R180"/>
+</instance>
 <instance part="JP1" gate="G$1" x="-12.7" y="76.2" rot="R180"/>
 <instance part="JP2" gate="G$1" x="91.44" y="68.58"/>
 <instance part="GND1" gate="1" x="-2.54" y="68.58"/>
 <instance part="P+1" gate="VCC" x="-2.54" y="81.28"/>
-<instance part="P+2" gate="VCC" x="58.42" y="48.26"/>
+<instance part="P+2" gate="VCC" x="58.42" y="48.26" smashed="yes">
+<attribute name="VALUE" x="56.134" y="48.768" size="1.778" layer="96"/>
+</instance>
 <instance part="GND2" gate="1" x="33.02" y="33.02"/>
-<instance part="D3" gate="G$1" x="78.74" y="68.58" rot="R90"/>
+<instance part="D3" gate="G$1" x="78.74" y="68.58" smashed="yes" rot="R90">
+<attribute name="NAME" x="77.47" y="72.1106" size="1.778" layer="95"/>
+<attribute name="VALUE" x="81.0514" y="71.12" size="1.778" layer="96" rot="R90"/>
+</instance>
 </instances>
 <busses>
@@
 <pinref part="IC1" gate="A" pin="THR"/>
 <wire x1="55.88" y1="48.26" x2="53.34" y2="48.26" width="0.1524" layer="91"/>
-<pinref part="R3" gate="G$1" pin="S"/>
+<pinref part="PR1" gate="G$1" pin="S"/>
 <junction x="30.48" y="60.96"/>
 <pinref part="C1" gate="G$1" pin="1"/>
@@
 <wire x1="33.02" y1="43.18" x2="33.02" y2="35.56" width="0.1524" layer="91"/>
 <junction x="33.02" y="35.56"/>
-<pinref part="Q1" gate="G$1" pin="E"/>
+<pinref part="Q1" gate="G$1" pin="S"/>
 <wire x1="78.74" y1="35.56" x2="78.74" y2="55.88" width="0.1524" layer="91"/>
 <wire x1="78.74" y1="35.56" x2="33.02" y2="35.56" width="0.1524" layer="91"/>
@@
 <net name="N$11" class="0">
 <segment>
-<pinref part="Q1" gate="G$1" pin="C"/>
+<pinref part="Q1" gate="G$1" pin="D"/>
 <pinref part="JP2" gate="G$1" pin="2"/>
-<wire x1="78.74" y1="66.04" x2="83.82" y2="66.04" width="0.1524" layer="91"/>
-<wire x1="83.82" y1="66.04" x2="88.9" y2="68.58" width="0.1524" layer="91"/>
+<wire x1="78.74" y1="66.04" x2="88.9" y2="66.04" width="0.1524" layer="91"/>
+<wire x1="88.9" y1="66.04" x2="88.9" y2="68.58" width="0.1524" layer="91"/>
 <pinref part="D3" gate="G$1" pin="A"/>
 <junction x="78.74" y="66.04"/>
@@
 <segment>
 <pinref part="D1" gate="G$1" pin="C"/>
-<pinref part="R3" gate="G$1" pin="A"/>
+<pinref part="PR1" gate="G$1" pin="A"/>
 <wire x1="20.32" y1="55.88" x2="25.4" y2="55.88" width="0.1524" layer="91"/>
 </segment>
@@
 <net name="N$3" class="0">
 <segment>
-<pinref part="R3" gate="G$1" pin="E"/>
+<pinref part="PR1" gate="G$1" pin="E"/>
 <pinref part="D2" gate="G$1" pin="A"/>
 <wire x1="25.4" y1="66.04" x2="20.32" y2="66.04" width="0.1524" layer="91"/>

Commit message: Description update
Parts:
- D1, D2, D3: value (none) -> LL4148
Changed lines of the file:
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@@
 <parts>
 <part name="IC1" library="adafruit" deviceset="*555" device="D" technology="NE"/>
-<part name="D1" library="diode" deviceset="DIODE-" device="MINIMELF"/>
-<part name="D2" library="diode" deviceset="DIODE-" device="MINIMELF"/>
+<part name="D1" library="diode" deviceset="DIODE-" device="MINIMELF" value="LL4148"/>
+<part name="D2" library="diode" deviceset="DIODE-" device="MINIMELF" value="LL4148"/>
 <part name="R1" library="rcl" deviceset="R-EU_" device="R0603" value="1K"/>
 <part name="R2" library="rcl" deviceset="R-EU_" device="R0603" value="47R"/>
@@
 <part name="P+2" library="supply1" deviceset="VCC" device=""/>
 <part name="GND2" library="supply1" deviceset="GND" device=""/>
-<part name="D3" library="diode" deviceset="DIODE-" device="MINIMELF"/>
+<part name="D3" library="diode" deviceset="DIODE-" device="MINIMELF" value="LL4148"/>
 </parts>
 <sheets>
@@
 <instance part="D1" gate="G$1" x="17.78" y="55.88" smashed="yes">
 <attribute name="NAME" x="11.684" y="54.8386" size="1.778" layer="95"/>
-<attribute name="VALUE" x="20.32" y="53.5686" size="1.778" layer="96"/>
+<attribute name="VALUE" x="11.43" y="52.2986" size="1.778" layer="96"/>
 </instance>
-<instance part="D2" gate="G$1" x="17.78" y="66.04" rot="R180"/>
+<instance part="D2" gate="G$1" x="17.78" y="66.04" smashed="yes" rot="R180">
+<attribute name="NAME" x="14.224" y="67.0814" size="1.778" layer="95" rot="R180"/>
+<attribute name="VALUE" x="5.08" y="62.9666" size="1.778" layer="96"/>
+</instance>
 <instance part="R1" gate="G$1" x="63.5" y="48.26" smashed="yes" rot="R90">
 <attribute name="NAME" x="65.024" y="49.2506" size="1.778" layer="95"/>
@@
 <instance part="GND2" gate="1" x="33.02" y="33.02"/>
 <instance part="D3" gate="G$1" x="78.74" y="68.58" smashed="yes" rot="R90">
-<attribute name="NAME" x="77.47" y="72.1106" size="1.778" layer="95"/>
-<attribute name="VALUE" x="81.0514" y="71.12" size="1.778" layer="96" rot="R90"/>
+<attribute name="NAME" x="72.898" y="68.5546" size="1.778" layer="95"/>
+<attribute name="VALUE" x="67.056" y="66.0146" size="1.778" layer="96"/>
 </instance>
 </instances>
